File: jtag_adapter/ft2232_jtag_tap.kicad_pcb (KiCad board)
At the start: 2 copper layers, 50 x 30 mm, 50 parts, among them J1 USB_C_Receptacle_USB2.0, J2 Conn_ARM_JTAG_SWD_20, U1 93AA56BT-I/OT, U2 FT232HL, Y1 Crystal_GND24

Commit message: v0.2に改修
Parts:
- removed D2: PGB1010603, Diode_SMD:D_0603_1608Metric
- removed R10: 10k, Resistor_SMD:R_0603_1608Metric
- removed R11, R12, R13, R14, R15, R16, R17: 0, Resistor_SMD:R_0603_1608Metric
- D1: value PGB1010603 -> PWR_LED; footprint Diode_SMD:D_0603_1608Metric -> LED_SMD:LED_0603_1608Metric
- J2: footprint Connector_PinHeader_2.54mm:PinHeader_2x10_P2.54mm_Horizontal -> Connector_IDC:IDC-Header_2x10_P2.54mm_Horizontal
- R7: value 0 -> 10k
- R8: value 0 -> 12k/1%
- R9: value 10k -> 1k
- moved R9 24.1 mm to (58.2, 104.3), turned to 0 degrees
- moved R7 18.0 mm to (80.1, 113.3), turned to 90 degrees
- moved D1 10.5 mm to (58.2, 102.8), turned to 180 degrees
- moved R6 6.71 mm to (64.0, 103.3), turned to 270 degrees
- moved C4 5.44 mm to (62.1, 107.5), turned to 180 degrees
- moved C5 4.94 mm to (62.1, 109.1), turned to 180 degrees
- moved R1 4.90 mm to (65.6, 103.3), turned to 270 degrees
- moved C16 4.61 mm to (77.8, 110.9), turned to 0 degrees
- moved L2 4.54 mm to (62.9, 112.2), turned to 90 degrees
- moved U1 3.93 mm to (70.4, 103.2)
- moved C9 3.68 mm to (64.4, 112.2), turned to 90 degrees
- moved R8 3.61 mm to (61.3, 112.2), turned to 270 degrees
- moved C1 3.57 mm to (67.2, 103.3), turned to 90 degrees
- moved R4 3.49 mm to (74.5, 103.9)
- moved R5 3.49 mm to (74.5, 102.3)
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Connections:
- C16 pad 2: GND -> GNDA
- D1 pad 1: Net-(D1-Pad1) -> GND
- D1 pad 2: GND -> Net-(D1-Pad2)
- J1 pad A6: Net-(D2-Pad1) -> /USB_D+
- J1 pad A7: Net-(D1-Pad1) -> /USB_D-
- J1 pad B6: Net-(D2-Pad1) -> /USB_D+
- J1 pad B7: Net-(D1-Pad1) -> /USB_D-
- R7 pad 1: /USB_D- -> Net-(C3-Pad1)
- R7 pad 2: Net-(D1-Pad1) -> +3V3
- R8 pad 1: /USB_D+ -> GND
- R8 pad 2: Net-(D2-Pad1) -> Net-(R8-Pad2)
- R9 pad 1: Net-(C3-Pad1) -> Net-(D1-Pad2)
- R9 pad 2: +3V3 -> +5V
- U2 pad 13: Net-(R11-Pad2) -> /SK_TCK
- U2 pad 14: Net-(R12-Pad2) -> /DO_TDI
- U2 pad 15: Net-(R13-Pad2) -> /DI_TDO
- U2 pad 16: Net-(R14-Pad2) -> /CS_TMS
- U2 pad 17: Net-(R15-Pad2) -> /~SRST
- U2 pad 18: Net-(R16-Pad2) -> /~TRST
- U2 pad 20: Net-(R17-Pad2) -> /RTCK
- U2 pad 49: GND -> (no net)
- U2 pad 5: Net-(R10-Pad2) -> Net-(R8-Pad2)
Routing:
- net GND: track 52.3 -> 259.4 mm, vias 107 -> 124
- net /~SRST: track 28.2 -> 47.1 mm
- net Net-(R10-Pad2): track 10.6 -> 0.00 mm, vias 2 -> 0
- net GNDA: track 10.5 -> 21.0 mm, vias 1 -> 3
- net +3V3: track 95.0 -> 84.7 mm, vias 8 -> 9
- net /DO_TDI: track 32.2 -> 23.2 mm, vias 0 -> 1
- net Net-(R8-Pad2): track 0.00 -> 7.47 mm
- net /~TRST: track 14.0 -> 20.8 mm, vias 1 -> 0
- net /CS_TMS: track 27.3 -> 20.8 mm
- net +5V: track 22.6 -> 28.9 mm
- net Net-(D1-Pad1): track 6.13 -> 0.00 mm
- net Net-(D2-Pad1): track 6.07 -> 0.00 mm, vias 1 -> 0
- net /USB_D+: track 5.60 -> 11.4 mm, vias 0 -> 1
- net /USB_D-: track 5.68 -> 11.5 mm, vias 0 -> 1
- net /SK_TCK: track 29.1 -> 23.6 mm, vias 0 -> 1
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- added copper zone on F.Cu, net /USB_D+
- added copper zone on F.Cu, net /USB_D-
Other:
- board text added: "PWR_LED"
- board text added: "jtag adapter v0.2(2021.07.17) @tnishinaga"
- board text removed: "jtag adapter v0.1(2021.05.15) @tnishinaga"

Commit message: Add panelize
Connections:
- U2 pad 49: (no net) -> GND
Routing:
- net GND: vias 124 -> 133
- net (no net): vias 9 -> 0
Changed lines of the file:
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@@
     (descr "Through hole IDC box header, 2x10, 2.54mm pitch, DIN 41651 / IEC 60603-13, double rows, https://docs.google.com/spreadsheets/d/16SsEcesNF15N3Lb4niX7dcUr-NY5_MFPQhobNuNppn4/edit#gid=0")
     (tags "Through hole horizontal IDC box header THT 2x10 2.54mm double row")
-    (fp_text reference J2 (at 6.215 -6.1) (layer F.SilkS)
+    (fp_text reference J2 (at -2.54 -1.8) (layer F.SilkS)
       (effects (font (size 1 1) (thickness 0.15)))
     )
     (fp_text value Conn_ARM_JTAG_SWD_20 (at 6.215 28.96) (layer F.Fab)
-      (effects (font (size 1 1) (thickness 0.15)))
-    )
-    (fp_text user %R (at 8.83 11.43 90) (layer F.Fab)
       (effects (font (size 1 1) (thickness 0.15)))
     )
@@
     (fp_line (start 4.38 9.38) (end 13.28 9.38) (layer F.Fab) (width 0.1))
     (fp_line (start 4.38 13.48) (end 13.28 13.48) (layer F.Fab) (width 0.1))
-    (fp_line (start 4.27 9.38) (end 13.39 9.38) (layer F.SilkS) (width 0.12))
-    (fp_line (start 4.27 13.48) (end 13.39 13.48) (layer F.SilkS) (width 0.12))
     (fp_line (start 4.38 -0.32) (end -0.32 -0.32) (layer F.Fab) (width 0.1))
     (fp_line (start -0.32 -0.32) (end -0.32 0.32) (layer F.Fab) (width 0.1))
@@
     (fp_line (start 13.28 27.96) (end 4.38 27.96) (layer F.Fab) (width 0.1))
     (fp_line (start 4.38 27.96) (end 4.38 -4.1) (layer F.Fab) (width 0.1))
-    (fp_line (start 4.27 -5.21) (end 13.39 -5.21) (layer F.SilkS) (width 0.12))
-    (fp_line (start 13.39 -5.21) (end 13.39 28.07) (layer F.SilkS) (width 0.12))
-    (fp_line (start 13.39 28.07) (end 4.27 28.07) (layer F.SilkS) (width 0.12))
-    (fp_line (start 4.27 28.07) (end 4.27 -5.21) (layer F.SilkS) (width 0.12))
     (fp_line (start -1.35 0) (end -2.35 -0.5) (layer F.SilkS) (width 0.12))
     (fp_line (start -2.35 -0.5) (end -2.35 0.5) (layer F.SilkS) (width 0.12))
@@
     (fp_line (start 13.78 28.46) (end 13.78 -5.6) (layer F.CrtYd) (width 0.05))
     (fp_line (start 13.78 -5.6) (end -1.35 -5.6) (layer F.CrtYd) (width 0.05))
+    (fp_text user %R (at 8.83 11.43 90) (layer F.Fab)
+      (effects (font (size 1 1) (thickness 0.15)))
+    )
     (pad 20 thru_hole circle (at 2.54 22.86) (size 1.7 1.7) (drill 1) (layers *.Cu *.Mask)
       (net 1 GND))
@@
     (pad "" smd roundrect (at -1.2 0) (size 0.97 0.97) (layers F.Paste) (roundrect_rratio 0.25))
     (pad "" smd roundrect (at -1.2 -1.2) (size 0.97 0.97) (layers F.Paste) (roundrect_rratio 0.25))
-    (pad 49 smd rect (at 0 0) (size 3.6 3.6) (layers F.Cu F.Mask))
+    (pad 49 smd rect (at 0 0) (size 3.6 3.6) (layers F.Cu F.Mask)
+      (net 1 GND))
     (pad 48 smd roundrect (at -2.75 -4.1625) (size 0.3 1.475) (layers F.Cu F.Paste F.Mask) (roundrect_rratio 0.25)
       (net 1 GND))
@@
   (gr_line (start 50 100) (end 100 100) (layer Edge.Cuts) (width 0.05))
   (gr_line (start 50 100) (end 50 130) (layer Edge.Cuts) (width 0.05))
-  (via (at 72.39 115.062) (size 0.6) (drill 0.3) (layers F.Cu B.Cu) (net 0))
-  (via (at 71.628 115.062) (size 0.6) (drill 0.3) (layers F.Cu B.Cu) (net 0))
-  (via (at 71.628 115.824) (size 0.6) (drill 0.3) (layers F.Cu B.Cu) (net 0))
-  (via (at 72.39 115.824) (size 0.6) (drill 0.3) (layers F.Cu B.Cu) (net 0))
-  (via (at 73.152 115.824) (size 0.6) (drill 0.3) (layers F.Cu B.Cu) (net 0))
-  (via (at 73.152 115.062) (size 0.6) (drill 0.3) (layers F.Cu B.Cu) (net 0))
-  (via (at 73.152 114.3) (size 0.6) (drill 0.3) (layers F.Cu B.Cu) (net 0))
-  (via (at 72.39 114.3) (size 0.6) (drill 0.3) (layers F.Cu B.Cu) (net 0))
-  (via (at 71.628 114.3) (size 0.6) (drill 0.3) (layers F.Cu B.Cu) (net 0))
+  (via (at 72.39 115.062) (size 0.6) (drill 0.3) (layers F.Cu B.Cu) (net 1))
+  (via (at 71.628 115.062) (size 0.6) (drill 0.3) (layers F.Cu B.Cu) (net 1))
+  (via (at 71.628 115.824) (size 0.6) (drill 0.3) (layers F.Cu B.Cu) (net 1))
+  (via (at 72.39 115.824) (size 0.6) (drill 0.3) (layers F.Cu B.Cu) (net 1))
+  (via (at 73.152 115.824) (size 0.6) (drill 0.3) (layers F.Cu B.Cu) (net 1))
+  (via (at 73.152 115.062) (size 0.6) (drill 0.3) (layers F.Cu B.Cu) (net 1))
+  (via (at 73.152 114.3) (size 0.6) (drill 0.3) (layers F.Cu B.Cu) (net 1))
+  (via (at 72.39 114.3) (size 0.6) (drill 0.3) (layers F.Cu B.Cu) (net 1))
+  (via (at 71.628 114.3) (size 0.6) (drill 0.3) (layers F.Cu B.Cu) (net 1))
   (via (at 72.68 103.24) (size 0.6) (drill 0.3) (layers F.Cu B.Cu) (net 1))
   (segment (start 71.51 103.24) (end 72.68 103.24) (width 0.25) (layer F.Cu) (net 1))
@@
   (via (at 68.326 105.156) (size 0.6) (drill 0.3) (layers F.Cu B.Cu) (net 1))
   (via (at 69.342 105.156) (size 0.6) (drill 0.3) (layers F.Cu B.Cu) (net 1))
-  (via (at 63.44 106.44) (size 0.6) (drill 0.3) (layers F.Cu B.Cu) (net 1))
+  (via (at 63.31 106.26) (size 0.6) (drill 0.3) (layers F.Cu B.Cu) (net 1))
   (via (at 81.28 110.998) (size 0.6) (drill 0.3) (layers F.Cu B.Cu) (net 1))
   (via (at 74.93 116.332) (size 0.6) (drill 0.3) (layers F.Cu B.Cu) (net 1))
@@
     (connect_pads (clearance 0.2))
     (min_thickness 0.127)
-    (fill (arc_segments 32) (thermal_gap 0.2) (thermal_bridge_width 0.2))
+    (fill yes (arc_segments 32) (thermal_gap 0.2) (thermal_bridge_width 0.2))
     (polygon
       (pts
@@
     (connect_pads (clearance 0.2))
     (min_thickness 0.127)
-    (fill (arc_segments 32) (thermal_gap 0.2) (thermal_bridge_width 0.2))
+    (fill yes (arc_segments 32) (thermal_gap 0.2) (thermal_bridge_width 0.2))
     (polygon
       (pts
@@
     (connect_pads yes (clearance 0.2))
     (min_thickness 0.2)
-    (fill (arc_segments 32) (thermal_gap 0.2) (thermal_bridge_width 0.3))
+    (fill yes (arc_segments 32) (thermal_gap 0.2) (thermal_bridge_width 0.3))
     (polygon
       (pts
@@
     (connect_pads yes (clearance 0.2))
     (min_thickness 0.2)
-    (fill (arc_segments 32) (thermal_gap 0.2) (thermal_bridge_width 0.3))
+    (fill yes (arc_segments 32) (thermal_gap 0.2) (thermal_bridge_width 0.3))
     (polygon
       (pts
