File: jtag_adapter/usb.sch (KiCad schematic (older format))
At the start: 9 parts, among them J1 USB_C_Receptacle_USB2.0

Commit message: wip
Parts:
- gave numbers to parts that had none: 3
- renumbered L1 to L2, R1 to R3, R2 to R4
Changed lines of the file:
@@
 encoding utf-8
 Sheet 2 4
-Title ""
-Date ""
-Rev ""
-Comp ""
+Title "FT232 JTAG adapter"
+Date "2021-09-01"
+Rev "v1.0"
+Comp "Toshifumi NISHINAGA(@tnishinaga)"
 Comment1 ""
 Comment2 ""
@@
 $EndComp
 $Comp
-L power:+5V #PWR0102
+L power:+5V #PWR013
 U 1 1 612382F4
 P 6150 2200
-F 0 "#PWR0102" H 6150 2050 50  0001 C CNN
+F 0 "#PWR013" H 6150 2050 50  0001 C CNN
 F 1 "+5V" H 6165 2373 50  0000 C CNN
 F 2 "" H 6150 2200 50  0001 C CNN
@@
 $EndComp
 $Comp
-L power:GND #PWR0103
+L power:GND #PWR011
 U 1 1 612382FA
 P 4750 4800
-F 0 "#PWR0103" H 4750 4550 50  0001 C CNN
+F 0 "#PWR011" H 4750 4550 50  0001 C CNN
 F 1 "GND" H 4755 4627 50  0000 C CNN
 F 2 "" H 4750 4800 50  0001 C CNN
@@
 	4450 4400 4450 4550
 $Comp
-L Device:R R1
+L Device:R R3
 U 1 1 61238308
 P 5700 3100
-F 0 "R1" V 5600 3200 50  0000 C CNN
+F 0 "R3" V 5600 3200 50  0000 C CNN
 F 1 "5.1k" V 5600 3000 50  0000 C CNN
 F 2 "Resistor_SMD:R_0603_1608Metric" V 5630 3100 50  0001 C CNN
@@
 $EndComp
 $Comp
-L Device:R R2
+L Device:R R4
 U 1 1 6123830F
 P 5700 3200
-F 0 "R2" V 5800 3300 50  0000 C CNN
+F 0 "R4" V 5800 3300 50  0000 C CNN
 F 1 "5.1k" V 5800 3100 50  0000 C CNN
 F 2 "Resistor_SMD:R_0603_1608Metric" V 5630 3200 50  0001 C CNN
@@
 $EndComp
 $Comp
-L power:GND #PWR0104
+L power:GND #PWR012
 U 1 1 61238315
 P 5950 3250
-F 0 "#PWR0104" H 5950 3000 50  0001 C CNN
+F 0 "#PWR012" H 5950 3000 50  0001 C CNN
 F 1 "GND" H 6050 3250 50  0000 C CNN
 F 2 "" H 5950 3250 50  0001 C CNN
@@
 $EndComp
 $Comp
-L power:GND #PWR0105
+L power:GND #PWR014
 U 1 1 61238334
 P 6150 3250
-F 0 "#PWR0105" H 6150 3000 50  0001 C CNN
+F 0 "#PWR014" H 6150 3000 50  0001 C CNN
 F 1 "GND" H 6250 3250 50  0000 C CNN
 F 2 "" H 6150 3250 50  0001 C CNN
@@
 Connection ~ 6150 2900
 $Comp
-L Device:L_Core_Ferrite L1
+L Device:L_Core_Ferrite L2
 U 1 1 6123833F
 P 6150 2550
-F 0 "L1" V 5969 2550 50  0000 C CNN
+F 0 "L2" V 5969 2550 50  0000 C CNN
 F 1 "600R/0.5A" V 6050 2550 50  0000 C CNN
 F 2 "Inductor_SMD:L_0603_1608Metric" H 6150 2550 50  0001 C CNN
@@
 D+
 $Comp
-L power:+5V #PWR0101
+L power:+5V #PWR09
 U 1 1 612DC969
 P 3000 2900
-F 0 "#PWR0101" H 3000 2750 50  0001 C CNN
+F 0 "#PWR09" H 3000 2750 50  0001 C CNN
 F 1 "+5V" H 3015 3073 50  0000 C CNN
 F 2 "" H 3000 2900 50  0001 C CNN
@@
 $EndComp
 $Comp
-L power:GND #PWR0141
+L power:GND #PWR010
 U 1 1 612DCF01
 P 3000 4250
-F 0 "#PWR0141" H 3000 4000 50  0001 C CNN
+F 0 "#PWR010" H 3000 4000 50  0001 C CNN
 F 1 "GND" H 3005 4077 50  0000 C CNN
 F 2 "" H 3000 4250 50  0001 C CNN
@@
 	4750 4400 4750 4550
 $Comp
-L Device:R R?
+L Device:R R2
 U 1 1 613D0918
 P 4600 4550
-F 0 "R?" V 4500 4650 50  0000 C CNN
+F 0 "R2" V 4500 4650 50  0000 C CNN
 F 1 "0" V 4500 4450 50  0000 C CNN
 F 2 "Resistor_SMD:R_0603_1608Metric" V 4530 4550 50  0001 C CNN
@@
 	4750 4550 4750 4800
 $Comp
-L Device:R R?
+L Device:R R5
 U 1 1 613D0CD8
 P 6000 3500
-F 0 "R?" V 5900 3600 50  0000 C CNN
+F 0 "R5" V 5900 3600 50  0000 C CNN
 F 1 "0" V 5900 3400 50  0000 C CNN
 F 2 "Resistor_SMD:R_0603_1608Metric" V 5930 3500 50  0001 C CNN
@@
 $EndComp
 $Comp
-L Device:R R?
+L Device:R R6
 U 1 1 613D16CD
 P 6000 3600
-F 0 "R?" V 6100 3700 50  0000 C CNN
+F 0 "R6" V 6100 3700 50  0000 C CNN
 F 1 "0" V 6100 3500 50  0000 C CNN
 F 2 "Resistor_SMD:R_0603_1608Metric" V 5930 3600 50  0001 C CNN

Commit message: wip
Parts:
- removed R2: 0, Resistor_SMD:R_0603_1608Metric, symbol Device:R
Connections:
- net +5V: no longer D2.4 (VCC)
- net GND: now also J1.S1 (SHIELD)
- net VBUS: now reaches C1.1, J1.A4 (VBUS), J1.A9 (VBUS), J1.B4 (VBUS), J1.B9 (VBUS), L2.2
- net VBUS: now also D2.4 (VCC)
Changed lines of the file:
@@
 D+
-$Comp
-L power:+5V #PWR09
-U 1 1 612DC969
-P 3000 2900
-F 0 "#PWR09" H 3000 2750 50  0001 C CNN
-F 1 "+5V" H 3015 3073 50  0000 C CNN
-F 2 "" H 3000 2900 50  0001 C CNN
-F 3 "" H 3000 2900 50  0001 C CNN
-	1    3000 2900
-	1    0    0    -1
-$EndComp
 $Comp
 L power:GND #PWR010
@@
 Wire Wire Line
 	6150 2200 6150 2400
-Wire Wire Line
-	4750 4400 4750 4550
-$Comp
-L Device:R R2
-U 1 1 613D0918
-P 4600 4550
-F 0 "R2" V 4500 4650 50  0000 C CNN
-F 1 "0" V 4500 4450 50  0000 C CNN
-F 2 "Resistor_SMD:R_0603_1608Metric" V 4530 4550 50  0001 C CNN
-F 3 "~" H 4600 4550 50  0001 C CNN
-F 4 "RC0603FR-075K1L" H 4600 4550 50  0001 C CNN "MPN"
-	1    4600 4550
-	0    1    1    0
-$EndComp
-Connection ~ 4750 4550
-Wire Wire Line
-	4750 4550 4750 4800
 $Comp
 L Device:R R5
@@
 Wire Wire Line
 	6550 3600 6150 3600
+Text Label 5500 2900 0    50   ~ 0
+VBUS
+Text Label 3000 2900 0    50   ~ 0
+VBUS
+Wire Wire Line
+	4750 4400 4750 4550
+Wire Wire Line
+	4450 4550 4750 4550
+Connection ~ 4750 4550
+Wire Wire Line
+	4750 4550 4750 4800
 $EndSCHEMATC
