File: jtag_adapter/jtag.sch (KiCad schematic (older format))
At the start: 15 parts, among them J2 Conn_ARM_JTAG_SWD_20, U3 SN74AXC2T45-Q1, U4 SN74AXC2T45-Q1, U5 SN74AXC2T45-Q1, U6 SN74AXC2T45-Q1

Commit message: wip
Parts:
- removed C20, C24, C25, C26: 0.1uF, Capacitor_SMD:C_0603_1608Metric, symbol Device:C
- removed R10, R11: 10k, Resistor_SMD:R_0603_1608Metric, symbol Device:R
- removed U3, U4, U5, U6: SN74AXC2T45-Q1, Package_SO:VSSOP-8_2.4x2.1mm_P0.5mm, symbol Logic_LevelTranslator:74LVC2T45DC
- added C21, C23: 0.1uF, Capacitor_SMD:C_0603_1608Metric, symbol Device:C
- added D4, D5: 1N4148W, Diode_SMD:D_SOD-123, symbol Device:D
- added Q1, Q2: BSS138, Package_TO_SOT_SMD:SOT-23, symbol Transistor_FET:BSS138
- added R15, R16, R17: 10k, Resistor_SMD:R_0603_1608Metric, symbol Device:R
- added R18, R19: 4.7k, Resistor_SMD:R_0603_1608Metric, symbol Device:R
- added R20, R21, R22, R23, R24, R25, R26: 0, Resistor_SMD:R_0603_1608Metric, symbol Device:R
- added U4, U5: SN74AXCH4T245PW, Package_SO:TSSOP-16_4.4x5mm_P0.65mm, symbol Logic_LevelTranslator:SN74AVC4T245PW
- added U6: SN74AXCH1T45, Package_TO_SOT_SMD:SOT-23-6, symbol Logic_LevelTranslator:SN74LVC1T45DBV
- renumbered C21 to C18, C23 to C20
Connections:
- net +3V3: now also R15.2, R18.2, R19.2, U4.1 (VCCA), U4.2 (1DIR), U5.1 (VCCA), U5.2 (1DIR), U6.6 (VCCB)
- net GND: now also C21.1, C23.1, R16.1, R17.2, U4.3 (2DIR), U4.8 (GND), U4.9 (GND), U5.3 (2DIR), U5.8 (GND), U5.9 (GND), U6.2 (GND), U6.5 (DIR)
- net JTAG_RTCK: now also U4.7 (2A2), U5.7 (2A2)
- net JTAG_TCK: now also U6.4 (B)
- net JTAG_TDI: now also U4.5 (1A2), U5.4 (1A1)
- net JTAG_TDO: now also U4.6 (2A1), U5.6 (2A1)
- net JTAG_TMS: now also U4.4 (1A1)
- net JTAG_~SRST: now also Q2.3 (D), R19.1
- net JTAG_~TRST: now also Q1.3 (D), R18.1
- net RTCK: now also R22.1, U4.10 (2B2); no longer J2.11 (RTCK)
- net TDI: now also R26.1, U4.12 (1B2); no longer J2.5 (TDI)
- net VTREF: now also C21.2, C23.2, Q1.1 (G), Q2.1 (G), U4.16 (VCCB), U5.16 (VCCB), U6.1 (VCCA)
- net ~SRST: now also Q2.2 (S), R21.1; no longer J2.15 (~SRST~)
- net ~TRST: now also Q1.2 (S), R20.1; no longer J2.3 (~TRST~)
- net TCK renamed CONN_TCK
- net CONN_TCK: now also R23.2
- net TDO renamed CONN_TDO
- net CONN_TDO: now also R25.2
- net TMS renamed CONN_TMS
- net CONN_TMS: now also R24.2
- new net: R17.1, U5.12 (1B2)
- new net: D4.2 (A), D5.2 (A), R15.1, U5.15 (1~OE)
- new net: R16.2, U5.5 (1A2)
- new net CONN_RTCK: J2.11 (RTCK), R22.2
- new net CONN_TDI: J2.5 (TDI), R26.2
- new net CONN_~SRST: J2.15 (~SRST~), R21.2
- new net CONN_~TRST: J2.3 (~TRST~), R20.2
- new net JTAG_EN: U4.14 (2~OE), U4.15 (1~OE)
- new net SWDIO_OE: D4.1 (K)
- new net SWD_EN: D5.1 (K), U5.14 (2~OE)
- new net TCK_SWDCLK: R23.1, U6.3 (A)
- new net TDO_SWO: R25.1, U4.11 (2B1), U5.10 (2B2)
- new net TMS_SWDIO: R24.1, U4.13 (1B1), U5.11 (2B1), U5.13 (1B1)
Other:
- note added: "1A -> 1B\n2A <- 2B\n"
- note added: "JTAG"
- note added: "SWD"
- note added: "common"
- moved on the sheet: C18, C20, J2

Commit message: wip
Parts:
- D4, D5: value 1N4148W -> CDSU101A; footprint Diode_SMD:D_SOD-123 -> Diode_SMD:D_SOD-523
Connections:
- net +3V3: now also U4.3 (2DIR), U5.3 (2DIR); no longer U4.2 (1DIR), U5.2 (1DIR)
- net GND: now also U4.2 (1DIR), U5.2 (1DIR); no longer U4.3 (2DIR), U5.3 (2DIR)
- net JTAG_RTCK: now also U4.5 (1A2), U5.5 (1A2); no longer U4.7 (2A2), U5.7 (2A2)
- net JTAG_TDI: now also U4.7 (2A2), U5.6 (2A1); no longer U4.5 (1A2), U5.4 (1A1)
- net JTAG_TDO: now also U4.4 (1A1), U5.4 (1A1); no longer U4.6 (2A1), U5.6 (2A1)
- net JTAG_TMS: now also U4.6 (2A1); no longer U4.4 (1A1)
- net RTCK: now also U4.12 (1B2); no longer U4.10 (2B2)
- net TDI: now also U4.10 (2B2); no longer U4.12 (1B2)
- net TDO_SWO: now also U4.13 (1B1), U5.12 (1B2); no longer U4.11 (2B1), U5.10 (2B2)
- net TMS_SWDIO: now also U4.11 (2B1); no longer U4.13 (1B1)
- net at R17.1: now also U5.10 (2B2); no longer U5.12 (1B2)
- net at R16.2: now also U5.7 (2A2); no longer U5.5 (1A2)
Other:
- note added: "1A <- 1B\n2A ->2B\n"
- note removed: "1A -> 1B\n2A <- 2B\n"
Changed lines of the file:
@@
 NoConn ~ 8900 4050
 NoConn ~ 9500 2750
-Text HLabel 1650 3250 0    50   Input ~ 0
+Text HLabel 1650 3050 0    50   Input ~ 0
 JTAG_RTCK
 Text HLabel 4700 5300 0    50   Input ~ 0
 JTAG_TCK
-Text HLabel 1650 3050 0    50   Input ~ 0
+Text HLabel 1650 3250 0    50   Input ~ 0
 JTAG_TDI
 Text Label 9600 2600 0    50   ~ 0
@@
 Text HLabel 1250 4600 0    50   Input ~ 0
 SWDIO_OE
-Text HLabel 1650 3150 0    50   Input ~ 0
+Text HLabel 1650 2950 0    50   Input ~ 0
 JTAG_TDO
 $Comp
@@
 	2050 2550 2150 2550
 Connection ~ 2050 2450
-Wire Wire Line
-	2150 2650 1800 2650
 $Comp
 L power:GND #PWR054
 U 1 1 6167DD42
-P 1800 2800
-F 0 "#PWR054" H 1800 2550 50  0001 C CNN
-F 1 "GND" H 1950 2750 50  0000 C CNN
-F 2 "" H 1800 2800 50  0001 C CNN
-F 3 "" H 1800 2800 50  0001 C CNN
-	1    1800 2800
-	1    0    0    -1
-$EndComp
-Wire Wire Line
-	2150 2750 1800 2750
+P 1950 2800
+F 0 "#PWR054" H 1950 2550 50  0001 C CNN
+F 1 "GND" H 2100 2750 50  0000 C CNN
+F 2 "" H 1950 2800 50  0001 C CNN
+F 3 "" H 1950 2800 50  0001 C CNN
+	1    1950 2800
+	1    0    0    -1
+$EndComp
 Wire Wire Line
 	2150 2950 1650 2950
@@
 	1650 3250 2150 3250
 Wire Wire Line
-	1800 2750 1800 2800
-Wire Wire Line
 	1650 2450 2050 2450
-Wire Wire Line
-	1800 2600 1800 2650
 Text Label 7250 3550 0    50   ~ 0
 TMS_SWDIO
-Text Label 3550 3250 0    50   ~ 0
+Text Label 3550 3050 0    50   ~ 0
 RTCK
 Text Label 5750 5300 0    50   ~ 0
 TCK_SWDCLK
+Text Label 3550 3150 0    50   ~ 0
+TMS_SWDIO
+Text HLabel 1650 3150 0    50   Input ~ 0
+JTAG_TMS
+Text Label 3550 3250 0    50   ~ 0
+TDI
 Text Label 3550 2950 0    50   ~ 0
-TMS_SWDIO
-Text HLabel 1650 2950 0    50   Input ~ 0
-JTAG_TMS
-Text Label 3550 3050 0    50   ~ 0
-TDI
-Text Label 3550 3150 0    50   ~ 0
 TDO_SWO
 Wire Wire Line
@@
 Wire Wire Line
 	2650 5850 2650 6000
-Wire Wire Line
-	2150 5050 1800 5050
 $Comp
 L power:GND #PWR056
 U 1 1 612EF461
-P 1800 5200
-F 0 "#PWR056" H 1800 4950 50  0001 C CNN
-F 1 "GND" H 1950 5150 50  0000 C CNN
-F 2 "" H 1800 5200 50  0001 C CNN
-F 3 "" H 1800 5200 50  0001 C CNN
-	1    1800 5200
-	1    0    0    -1
-$EndComp
-Wire Wire Line
-	2150 5150 1800 5150
+P 1950 5200
+F 0 "#PWR056" H 1950 4950 50  0001 C CNN
+F 1 "GND" H 2100 5150 50  0000 C CNN
+F 2 "" H 1950 5200 50  0001 C CNN
+F 3 "" H 1950 5200 50  0001 C CNN
+	1    1950 5200
+	1    0    0    -1
+$EndComp
+Wire Wire Line
+	2150 5550 1650 5550
 Wire Wire Line
 	2150 5350 1650 5350
 Wire Wire Line
-	2150 5550 1650 5550
-Wire Wire Line
-	1650 5650 2150 5650
-Wire Wire Line
-	1800 5150 1800 5200
-Wire Wire Line
-	1800 5000 1800 5050
+	1650 5450 2150 5450
+Wire Wire Line
+	3150 5550 3550 5550
 Wire Wire Line
 	3150 5350 3550 5350
 Wire Wire Line
-	3150 5550 3550 5550
-Wire Wire Line
-	3550 5650 3150 5650
+	3550 5450 3150 5450
 $Comp
 L power:+3.3V #PWR062
@@
 $EndComp
 Text Notes 3100 2700 0    50   ~ 0
-1A -> 1B\n2A <- 2B\n
-Text Notes 3100 5100 0    50   ~ 0
-1A -> 1B\n2A <- 2B\n
+1A <- 1B\n2A ->2B\n
+Text Label 3550 5550 0    50   ~ 0
+TMS_SWDIO
 Text Label 3550 5350 0    50   ~ 0
 TMS_SWDIO
-Text Label 3550 5550 0    50   ~ 0
-TMS_SWDIO
-Text Label 3550 5650 0    50   ~ 0
+Text Label 3550 5450 0    50   ~ 0
 TDO_SWO
+Text HLabel 1650 5350 0    50   Input ~ 0
+JTAG_TDO
+Text HLabel 1650 5450 0    50   Input ~ 0
+JTAG_RTCK
 Text HLabel 1650 5550 0    50   Input ~ 0
-JTAG_TDO
-Text HLabel 1650 5650 0    50   Input ~ 0
-JTAG_RTCK
-Text HLabel 1650 5350 0    50   Input ~ 0
 JTAG_TDI
 Wire Wire Line
@@
 P 1500 4600
 F 0 "D4" H 1350 4650 50  0000 C CNN
-F 1 "1N4148W" H 1750 4650 50  0000 C CNN
-F 2 "Diode_SMD:D_SOD-123" H 1500 4600 50  0001 C CNN
+F 1 "CDSU101A" H 1750 4650 50  0000 C CNN
+F 2 "Diode_SMD:D_SOD-523" H 1500 4600 50  0001 C CNN
 F 3 "~" H 1500 4600 50  0001 C CNN
 	1    1500 4600
@@
 P 1500 4750
 F 0 "D5" H 1350 4800 50  0000 C CNN
-F 1 "1N4148W" H 1750 4800 50  0000 C CNN
-F 2 "Diode_SMD:D_SOD-123" H 1500 4750 50  0001 C CNN
+F 1 "CDSU101A" H 1750 4800 50  0000 C CNN
+F 2 "Diode_SMD:D_SOD-523" H 1500 4750 50  0001 C CNN
 F 3 "~" H 1500 4750 50  0001 C CNN
 	1    1500 4750
@@
 	1    0    0    -1
 $EndComp
-Wire Wire Line
-	3150 5450 3250 5450
-Wire Wire Line
-	3250 5450 3250 5700
 $Comp
 L power:+3.3V #PWR057
@@
 	-1   0    0    1
 $EndComp
-Wire Wire Line
-	2150 5450 2050 5450
-Wire Wire Line
-	2050 5450 2050 5700
 Wire Wire Line
 	1300 4750 1300 4850
@@
 Wire Wire Line
 	7900 3050 7250 3050
+Wire Wire Line
+	2150 2650 1950 2650
+Wire Wire Line
+	1950 2650 1950 2800
+Wire Wire Line
+	2150 2750 1800 2750
+Wire Wire Line
+	1800 2750 1800 2600
+Text Notes 3150 5050 0    50   ~ 0
+1A <- 1B\n2A ->2B\n
+Wire Wire Line
+	2150 5150 1800 5150
+Wire Wire Line
+	1800 5150 1800 5000
+Wire Wire Line
+	2150 5050 1950 5050
+Wire Wire Line
+	1950 5050 1950 5200
+Wire Wire Line
+	2150 5650 2050 5650
+Wire Wire Line
+	2050 5650 2050 5700
+Wire Wire Line
+	3250 5650 3250 5700
+Wire Wire Line
+	3150 5650 3250 5650
 $EndSCHEMATC

Commit message: v1.0 基板発注
Parts:
- R18, R19: value 4.7k -> 10k
- U4, U5: MPN (none) -> SN74AXCH4T245PW
- U6: value SN74AXCH1T45 -> SN74AXCH1T45DBVR; MPN (none) -> SN74AXCH1T45DBVR
Connections:
- net +3V3: now also U4.2 (1DIR); no longer R18.2, R19.2, U4.3 (2DIR)
- net GND: now also U4.3 (2DIR); no longer U4.2 (1DIR)
- net JTAG_RTCK: now also U4.6 (2A1), U5.4 (1A1); no longer U4.5 (1A2), U5.5 (1A2)
- net JTAG_TDI: now also U4.4 (1A1); no longer U4.7 (2A2)
- net JTAG_TDO: now also U4.7 (2A2), U5.5 (1A2); no longer U4.4 (1A1), U5.4 (1A1)
- net JTAG_TMS: now also U4.5 (1A2); no longer U4.6 (2A1)
- net JTAG_~SRST: no longer R19.1
- net JTAG_~TRST: no longer R18.1
- net RTCK: now also U4.11 (2B1); no longer U4.12 (1B2)
- net TDI: now also U4.13 (1B1); no longer U4.10 (2B2)
- net TDO_SWO: now also U4.10 (2B2), U5.13 (1B1); no longer U4.13 (1B1), U5.12 (1B2)
- net TMS_SWDIO: now also U4.12 (1B2), U5.12 (1B2); no longer U4.11 (2B1), U5.13 (1B1)
- net VTREF: now also R18.2, R19.2
- net ~SRST: now also R19.1
- net ~TRST: now also R18.1
Other:
- note added: "1A -> 1B\n2A <- 2B\n"
- moved on the sheet: R18, R19
Changed lines of the file:
@@
 NoConn ~ 8900 4050
 NoConn ~ 9500 2750
-Text HLabel 1650 3050 0    50   Input ~ 0
+Text HLabel 1650 3150 0    50   Input ~ 0
 JTAG_RTCK
 Text HLabel 4700 5300 0    50   Input ~ 0
 JTAG_TCK
-Text HLabel 1650 3250 0    50   Input ~ 0
+Text HLabel 1650 2950 0    50   Input ~ 0
 JTAG_TDI
 Text Label 9600 2600 0    50   ~ 0
@@
 P 5200 5300
 F 0 "U6" H 5450 4950 50  0000 L CNN
-F 1 "SN74AXCH1T45" H 5350 4850 50  0000 L CNN
+F 1 "SN74AXCH1T45DBVR" H 5350 4850 50  0000 L CNN
 F 2 "Package_TO_SOT_SMD:SOT-23-6" H 5200 4850 50  0001 C CNN
 F 3 "" H 4300 4650 50  0001 C CNN
+F 4 "SN74AXCH1T45DBVR" H 5200 5300 50  0001 C CNN "MPN"
 	1    5200 5300
 	-1   0    0    -1
@@
 Text HLabel 1250 4600 0    50   Input ~ 0
 SWDIO_OE
-Text HLabel 1650 2950 0    50   Input ~ 0
+Text HLabel 1650 3250 0    50   Input ~ 0
 JTAG_TDO
 $Comp
@@
 Text Label 5600 2600 0    50   ~ 0
 ~TRST
-$Comp
-L power:+3.3V #PWR069
-U 1 1 61369BA3
-P 4950 2150
-F 0 "#PWR069" H 4950 2000 50  0001 C CNN
-F 1 "+3.3V" H 4965 2323 50  0000 C CNN
-F 2 "" H 4950 2150 50  0001 C CNN
-F 3 "" H 4950 2150 50  0001 C CNN
-	1    4950 2150
-	1    0    0    -1
-$EndComp
 Text HLabel 4900 3550 0    50   Input ~ 0
 JTAG_~SRST
@@
 L Device:R R?
 U 1 1 6152EABC
-P 4950 2400
+P 5550 2400
 AR Path="/6152EABC" Ref="R?"  Part="1"
 AR Path="/613347ED/6152EABC" Ref="R18"  Part="1"
-F 0 "R18" H 5100 2350 50  0000 C CNN
-F 1 "4.7k" H 5100 2450 50  0000 C CNN
-F 2 "Resistor_SMD:R_0603_1608Metric" V 4880 2400 50  0001 C CNN
-F 3 "~" H 4950 2400 50  0001 C CNN
-F 4 "" H 4950 2400 50  0001 C CNN "MPN"
-	1    4950 2400
+F 0 "R18" H 5700 2350 50  0000 C CNN
+F 1 "10k" H 5700 2450 50  0000 C CNN
+F 2 "Resistor_SMD:R_0603_1608Metric" V 5480 2400 50  0001 C CNN
+F 3 "~" H 5550 2400 50  0001 C CNN
+F 4 "" H 5550 2400 50  0001 C CNN "MPN"
+	1    5550 2400
 	-1   0    0    1
 $EndComp
 Wire Wire Line
-	5250 2050 5250 2300
-Wire Wire Line
-	5450 2600 5600 2600
+	5250 2050 5250 2150
+Wire Wire Line
+	5450 2600 5550 2600
 Text Label 5300 3000 0    50   ~ 0
 VTREF
 $Comp
-L power:+3.3V #PWR070
-U 1 1 61545718
-P 5000 3100
-F 0 "#PWR070" H 5000 2950 50  0001 C CNN
-F 1 "+3.3V" H 5015 3273 50  0000 C CNN
-F 2 "" H 5000 3100 50  0001 C CNN
-F 3 "" H 5000 3100 50  0001 C CNN
-	1    5000 3100
-	1    0    0    -1
-$EndComp
-$Comp
-L Transistor_FET:BSS138 Q2
-U 1 1 6154571F
-P 5300 3450
-F 0 "Q2" V 5500 3700 50  0000 C CNN
-F 1 "BSS138" V 5500 3200 50  0000 C CNN
-F 2 "Package_TO_SOT_SMD:SOT-23" H 5500 3375 50  0001 L CIN
-F 3 "https://www.onsemi.com/pub/Collateral/BSS138-D.PDF" H 5300 3450 50  0001 L CNN
-	1    5300 3450
-	0    -1   1    0
-$EndComp
-$Comp
 L Device:R R?
 U 1 1 61545726
-P 5000 3350
+P 5600 3350
 AR Path="/61545726" Ref="R?"  Part="1"
 AR Path="/613347ED/61545726" Ref="R19"  Part="1"
-F 0 "R19" H 5150 3300 50  0000 C CNN
-F 1 "4.7k" H 5150 3400 50  0000 C CNN
-F 2 "Resistor_SMD:R_0603_1608Metric" V 4930 3350 50  0001 C CNN
-F 3 "~" H 5000 3350 50  0001 C CNN
-F 4 "" H 5000 3350 50  0001 C CNN "MPN"
-	1    5000 3350
+F 0 "R19" H 5750 3300 50  0000 C CNN
+F 1 "10k" H 5750 3400 50  0000 C CNN
+F 2 "Resistor_SMD:R_0603_1608Metric" V 5530 3350 50  0001 C CNN
+F 3 "~" H 5600 3350 50  0001 C CNN
+F 4 "" H 5600 3350 50  0001 C CNN "MPN"
+	1    5600 3350
 	-1   0    0    1
 $EndComp
 Wire Wire Line
-	5300 3000 5300 3250
-Wire Wire Line
-	5500 3550 5650 3550
-Wire Wire Line
-	4900 3550 5000 3550
-Wire Wire Line
-	4850 2600 4950 2600
-Wire Wire Line
-	4950 2550 4950 2600
-Connection ~ 4950 2600
-Wire Wire Line
-	4950 2600 5050 2600
-Wire Wire Line
-	4950 2250 4950 2150
-Wire Wire Line
-	5000 3200 5000 3100
-Wire Wire Line
-	5000 3500 5000 3550
-Connection ~ 5000 3550
-Wire Wire Line
-	5000 3550 5100 3550
+	5300 3000 5300 3150
+Wire Wire Line
+	5500 3550 5600 3550
 $Comp
 L power:GND #PWR?
@@
 F 2 "Package_SO:TSSOP-16_4.4x5mm_P0.65mm" H 2650 2750 50  0001 C CNN
 F 3 "" H 2600 2600 50  0001 C CNN
+F 4 "SN74AXCH4T245PW" H 2650 2850 50  0001 C CNN "MPN"
 	1    2650 2850
 	1    0    0    -1
@@
 Text Label 7250 3550 0    50   ~ 0
 TMS_SWDIO
-Text Label 3550 3050 0    50   ~ 0
+Text Label 3550 3150 0    50   ~ 0
 RTCK
 Text Label 5750 5300 0    50   ~ 0
 TCK_SWDCLK
-Text Label 3550 3150 0    50   ~ 0
+Text Label 3550 3050 0    50   ~ 0
 TMS_SWDIO
-Text HLabel 1650 3150 0    50   Input ~ 0
+Text HLabel 1650 3050 0    50   Input ~ 0
 JTAG_TMS
+Text Label 3550 2950 0    50   ~ 0
+TDI
 Text Label 3550 3250 0    50   ~ 0
-TDI
-Text Label 3550 2950 0    50   ~ 0
 TDO_SWO
 Wire Wire Line
@@
 F 2 "Package_SO:TSSOP-16_4.4x5mm_P0.65mm" H 2650 5150 50  0001 C CNN
 F 3 "" H 2600 5000 50  0001 C CNN
+F 4 "SN74AXCH4T245PW" H 2650 5250 50  0001 C CNN "MPN"
 	1    2650 5250
 	1    0    0    -1
@@
 	1    0    0    -1
 $EndComp
-Text Notes 3100 2700 0    50   ~ 0
-1A <- 1B\n2A ->2B\n
 Text Label 3550 5550 0    50   ~ 0
 TMS_SWDIO
+Text Label 3550 5450 0    50   ~ 0
+TMS_SWDIO
 Text Label 3550 5350 0    50   ~ 0
-TMS_SWDIO
-Text Label 3550 5450 0    50   ~ 0
 TDO_SWO
+Text HLabel 1650 5450 0    50   Input ~ 0
+JTAG_TDO
 Text HLabel 1650 5350 0    50   Input ~ 0
-JTAG_TDO
-Text HLabel 1650 5450 0    50   Input ~ 0
 JTAG_RTCK
 Text HLabel 1650 5550 0    50   Input ~ 0
@@
 Wire Wire Line
 	7900 3050 7250 3050
-Wire Wire Line
-	2150 2650 1950 2650
-Wire Wire Line
-	1950 2650 1950 2800
-Wire Wire Line
-	2150 2750 1800 2750
-Wire Wire Line
-	1800 2750 1800 2600
 Text Notes 3150 5050 0    50   ~ 0
 1A <- 1B\n2A ->2B\n
@@
 Wire Wire Line
 	3150 5650 3250 5650
+$Comp
+L Transistor_FET:BSS138 Q2
+U 1 1 6154571F
+P 5300 3450
+F 0 "Q2" V 5500 3700 50  0000 C CNN
+F 1 "BSS138" V 5500 3200 50  0000 C CNN
+F 2 "Package_TO_SOT_SMD:SOT-23" H 5500 3375 50  0001 L CIN
+F 3 "https://www.onsemi.com/pub/Collateral/BSS138-D.PDF" H 5300 3450 50  0001 L CNN
+	1    5300 3450
+	0    -1   1    0
+$EndComp
+Wire Wire Line
+	4850 2600 5050 2600
+Wire Wire Line
+	4900 3550 5100 3550
+Wire Wire Line
+	5250 2150 5550 2150
+Wire Wire Line
+	5550 2150 5550 2250
+Connection ~ 5250 2150
+Wire Wire Line
+	5250 2150 5250 2300
+Wire Wire Line
+	5550 2550 5550 2600
+Connection ~ 5550 2600
+Wire Wire Line
+	5550 2600 5600 2600
+Wire Wire Line
+	5600 3500 5600 3550
+Connection ~ 5600 3550
+Wire Wire Line
+	5600 3550 5650 3550
+Wire Wire Line
+	5600 3200 5600 3150
+Wire Wire Line
+	5600 3150 5300 3150
+Connection ~ 5300 3150
+Wire Wire Line
+	5300 3150 5300 3250
+Wire Wire Line
+	1950 2800 1950 2750
+Wire Wire Line
+	1950 2750 2150 2750
+Wire Wire Line
+	2150 2650 1800 2650
+Wire Wire Line
+	1800 2650 1800 2600
+Text Notes 3100 2700 0    50   ~ 0
+1A -> 1B\n2A <- 2B\n
 $EndSCHEMATC
